File: KiCad/FencingTester.kicad_pcb (KiCad board)
At the start: 2 copper layers, 114.5 x 60.5 mm, 96 parts, among them IC1 ATMEGA328P-P, P1 SERIAL, P2 CONN_01X03, P3 CONN_01X03, P4 USB_OTG, Q1 Q_NMOS_GSD, Q10 Q_NMOS_GSD, Q11 Q_PMOS_DGS, Q12 Q_NMOS_GSD, Q2 Q_NMOS_GSD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

Commit message: Wiring PCB
Routing:
- net Net-(D13-Pad1): track 4.26 -> 37.3 mm
- net Net-(Q10-Pad1): track 0.18 -> 31.0 mm
- net /bargraph_driver/L10: track 4.26 -> 22.5 mm
- net Net-(D10-Pad1): track 8.73 -> 16.3 mm
- net /bargraph_driver/L9: track 6.94 -> 13.4 mm
Changed lines of the file:
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@@
     (thickness 1.6)
     (drawings 34)
-    (tracks 655)
+    (tracks 687)
     (zones 0)
     (modules 96)
@@
   (segment (start 175.26 46.99) (end 175.26 47.88) (width 0.25) (layer F.Cu) (net 9))
   (segment (start 176.53 45.72) (end 175.26 46.99) (width 0.25) (layer F.Cu) (net 9))
-  (segment (start 182.351 63.576) (end 179.735 60.96) (width 0.25) (layer F.Cu) (net 9))
-  (segment (start 182.351 64.276) (end 182.351 63.576) (width 0.25) (layer F.Cu) (net 9))
-  (segment (start 179.735 60.96) (end 175.895 60.96) (width 0.25) (layer F.Cu) (net 9))
-  (segment (start 175.895 60.96) (end 172.72 57.785) (width 0.25) (layer F.Cu) (net 9))
-  (segment (start 172.72 57.785) (end 172.72 48.895) (width 0.25) (layer F.Cu) (net 9))
-  (segment (start 173.735 47.88) (end 175.26 47.88) (width 0.25) (layer F.Cu) (net 9))
-  (segment (start 172.72 48.895) (end 173.735 47.88) (width 0.25) (layer F.Cu) (net 9))
+  (segment (start 175.26 47.88) (end 173.735 47.88) (width 0.25) (layer F.Cu) (net 9))
+  (segment (start 173.735 47.88) (end 173.355 48.26) (width 0.25) (layer F.Cu) (net 9))
+  (segment (start 173.355 48.26) (end 173.355 52.07) (width 0.25) (layer F.Cu) (net 9))
+  (segment (start 173.355 52.07) (end 175.26 53.975) (width 0.25) (layer F.Cu) (net 9))
+  (segment (start 175.26 53.975) (end 177.165 53.975) (width 0.25) (layer F.Cu) (net 9))
+  (segment (start 178.024999 54.834999) (end 178.024999 59.914999) (width 0.25) (layer F.Cu) (net 9))
+  (segment (start 177.165 53.975) (end 178.024999 54.834999) (width 0.25) (layer F.Cu) (net 9))
+  (segment (start 178.024999 59.914999) (end 179.07 60.96) (width 0.25) (layer F.Cu) (net 9))
+  (segment (start 179.07 60.96) (end 181.61 60.96) (width 0.25) (layer F.Cu) (net 9))
+  (segment (start 182.351 61.701) (end 182.351 64.276) (width 0.25) (layer F.Cu) (net 9))
+  (segment (start 181.61 60.96) (end 182.351 61.701) (width 0.25) (layer F.Cu) (net 9))
   (segment (start 188.701 64.276) (end 188.701 62.759) (width 0.25) (layer F.Cu) (net 10))
   (segment (start 191.8 59.66) (end 191.8 56.83) (width 0.25) (layer F.Cu) (net 10))
   (segment (start 188.701 62.759) (end 191.8 59.66) (width 0.25) (layer F.Cu) (net 10))
+  (segment (start 191.8 56.83) (end 193.36 56.83) (width 0.25) (layer F.Cu) (net 10))
+  (segment (start 194.31 51.88) (end 194.31 51.18) (width 0.25) (layer F.Cu) (net 10))
+  (segment (start 193.36 52.83) (end 194.31 51.88) (width 0.25) (layer F.Cu) (net 10))
+  (segment (start 193.36 56.83) (end 193.36 52.83) (width 0.25) (layer F.Cu) (net 10))
   (segment (start 198.15 47.85) (end 198.12 47.88) (width 0.25) (layer F.Cu) (net 11))
   (segment (start 198.15 44.13) (end 198.15 47.85) (width 0.25) (layer F.Cu) (net 11))
@@
   (segment (start 204.5 44.13) (end 204.5 44.78) (width 0.25) (layer F.Cu) (net 13))
   (segment (start 205.74 46.02) (end 205.74 47.88) (width 0.25) (layer F.Cu) (net 13))
+  (segment (start 204.215 47.88) (end 205.74 47.88) (width 0.25) (layer F.Cu) (net 13))
+  (segment (start 203.835 48.26) (end 204.215 47.88) (width 0.25) (layer F.Cu) (net 13))
+  (segment (start 203.2 52.705) (end 203.835 52.07) (width 0.25) (layer F.Cu) (net 13))
+  (segment (start 202.565 52.705) (end 203.2 52.705) (width 0.25) (layer F.Cu) (net 13))
+  (segment (start 191.241 72.426) (end 194.945 68.722) (width 0.25) (layer F.Cu) (net 13))
+  (segment (start 194.945 68.722) (end 194.945 65.405) (width 0.25) (layer F.Cu) (net 13))
+  (segment (start 203.835 52.07) (end 203.835 48.26) (width 0.25) (layer F.Cu) (net 13))
+  (segment (start 191.241 73.676) (end 191.241 72.426) (width 0.25) (layer F.Cu) (net 13))
+  (segment (start 194.945 65.405) (end 200.66 59.69) (width 0.25) (layer F.Cu) (net 13))
+  (segment (start 200.66 59.69) (end 200.66 54.61) (width 0.25) (layer F.Cu) (net 13))
+  (segment (start 200.66 54.61) (end 202.565 52.705) (width 0.25) (layer F.Cu) (net 13))
   (segment (start 123.5 40.655) (end 136.05 40.655) (width 0.4) (layer B.Cu) (net 14))
   (segment (start 137.955 24.78) (end 137.955 38.75) (width 0.4) (layer F.Cu) (net 14))
@@
   (segment (start 199.39 40.64) (end 199.39 39.465) (width 0.25) (layer F.Cu) (net 72))
   (segment (start 200.66 41.91) (end 199.39 40.64) (width 0.25) (layer F.Cu) (net 72))
+  (segment (start 200.66 41.91) (end 200.66 44.45) (width 0.4) (layer F.Cu) (net 72))
+  (segment (start 200.66 44.45) (end 201.93 45.72) (width 0.4) (layer F.Cu) (net 72))
+  (segment (start 201.93 45.72) (end 201.93 47.88) (width 0.4) (layer F.Cu) (net 72))
   (segment (start 205.74 51.18) (end 205.74 52.07) (width 0.25) (layer F.Cu) (net 73))
   (segment (start 204.5 53.31) (end 204.5 54.93) (width 0.25) (layer F.Cu) (net 73))
   (segment (start 205.74 52.07) (end 204.5 53.31) (width 0.25) (layer F.Cu) (net 73))
+  (segment (start 206.74 51.18) (end 208.28 49.64) (width 0.4) (layer F.Cu) (net 73))
+  (segment (start 205.74 51.18) (end 206.74 51.18) (width 0.4) (layer F.Cu) (net 73))
+  (segment (start 208.28 49.64) (end 208.28 41.91) (width 0.4) (layer F.Cu) (net 73))
+  (segment (start 205.835 39.465) (end 201.93 39.465) (width 0.4) (layer F.Cu) (net 73))
+  (segment (start 208.28 41.91) (end 205.835 39.465) (width 0.4) (layer F.Cu) (net 73))
   (segment (start 189.971 72.913) (end 190.098 73.04) (width 0.25) (layer F.Cu) (net 74) (status 30))
+  (segment (start 189.971 73.676) (end 189.971 75.036) (width 0.25) (layer F.Cu) (net 74))
+  (segment (start 189.971 75.036) (end 190.5 75.565) (width 0.25) (layer F.Cu) (net 74))
+  (segment (start 190.5 75.565) (end 198.12 75.565) (width 0.25) (layer F.Cu) (net 74))
+  (segment (start 198.12 75.565) (end 204.47 69.215) (width 0.25) (layer F.Cu) (net 74))
+  (segment (start 204.47 69.215) (end 204.47 57.15) (width 0.25) (layer F.Cu) (net 74))
   (segment (start 122.28 64.912) (end 120.792 64.912) (width 0.4) (layer B.Cu) (net 75))
   (segment (start 129.9 64.912) (end 122.28 64.912) (width 0.4) (layer B.Cu) (net 75))

Commit message: Importing new netlist
Parts:
- removed C8: 10µF, Capacitors_SMD:C_0805_HandSoldering
- removed D10, D11, D12, D13, D5, D6, D7, D8, D9: D_Small, Diodes_SMD:D_SOD-123
- removed Q1, Q10, Q12, Q2, Q3, Q4, Q5, Q6, Q7, Q8, Q9: Q_NMOS_GSD, custom-fencingTester:TSMT3
- removed Q11: Q_PMOS_DGS, custom-fencingTester:TSOP-6_HandSoldering
- removed R17, R18, R19, R20, R21, R22, R23, R24, R25: 330, Resistors_SMD:R_0805_HandSoldering
- removed R29: 2k, Resistors_SMD:R_0805_HandSoldering
- removed R46: 10k, Resistors_SMD:R_0805_HandSoldering
- R15: value 330 -> R
- R16: value 330 -> 10k
- U1: value CD74HC4067 -> TLC59116; footprint Housings_SOIC:SOIC-24W_7.5x15.4mm_Pitch1.27mm -> Housings_SSOP:TSSOP-28_4.4x9.7mm_Pitch0.65mm
- moved R15 47.9 mm to (218.8, 60.7)
- moved R16 43.6 mm to (213.4, 65.0)
- moved D4 23.0 mm to (199.2, 21.9), turned to 270 degrees
- moved U1 21.5 mm to (189.9, 47.9)
Connections:
- AR1 pad 1: +5V -> Net-(AR1-Pad1)
- C5 pad 2: +5V -> Net-(AR1-Pad1)
- D16 pad 1: Net-(D16-Pad1) -> (no net)
- D16 pad 2: Net-(D16-Pad2) -> (no net)
- D4 pad 10: Net-(D4-Pad10) -> +5V
- D4 pad 12: Net-(D4-Pad12) -> +5V
- D4 pad 13: Net-(D4-Pad13) -> +5V
- D4 pad 14: Net-(D4-Pad14) -> +5V
- D4 pad 15: Net-(D4-Pad15) -> +5V
- D4 pad 17: Net-(D4-Pad17) -> +5V
- D4 pad 19: Net-(D4-Pad19) -> +5V
- D4 pad 2: Net-(D4-Pad2) -> +5V
- D4 pad 21: GND -> Net-(D4-Pad21)
- D4 pad 22: GND -> Net-(D4-Pad22)
- D4 pad 23: GND -> Net-(D4-Pad23)
- D4 pad 24: GND -> Net-(D4-Pad24)
- D4 pad 25: GND -> Net-(D4-Pad25)
- D4 pad 26: GND -> Net-(D4-Pad26)
- D4 pad 27: GND -> Net-(D4-Pad27)
- D4 pad 28: GND -> Net-(D4-Pad28)
- D4 pad 29: GND -> Net-(D4-Pad29)
- D4 pad 30: GND -> Net-(D4-Pad30)
- D4 pad 4: Net-(D4-Pad4) -> +5V
- D4 pad 6: Net-(D4-Pad6) -> +5V
- D4 pad 8: Net-(D4-Pad8) -> +5V
- F1 pad 2: /power rail/BSense -> /BSense
- IC1 pad 11: /bargraph_driver/S3 -> (no net)
- IC1 pad 21: Net-(IC1-Pad21) -> (no net)
- IC1 pad 24: Net-(IC1-Pad24) -> /BSense
- IC1 pad 25: Net-(IC1-Pad25) -> (no net)
- IC1 pad 26: Net-(IC1-Pad26) -> (no net)
- IC1 pad 27: /power rail/BSense -> /SDA
- IC1 pad 28: Net-(IC1-Pad28) -> /SCL
- IC1 pad 4: /bargraph_driver/S0 -> Net-(IC1-Pad4)
- IC1 pad 5: /bargraph_driver/S1 -> Net-(IC1-Pad5)
- IC1 pad 6: /bargraph_driver/S2 -> Net-(IC1-Pad6)
- P1 pad 2: Net-(P1-Pad2) -> (no net)
- P4 pad 2: Net-(P4-Pad2) -> (no net)
- P4 pad 3: Net-(P4-Pad3) -> (no net)
- P4 pad 4: Net-(P4-Pad4) -> (no net)
- R15 pad 1: Net-(D4-Pad2) -> Net-(R15-Pad1)
- R15 pad 2: /bargraph_driver/L1 -> GND
- R16 pad 1: Net-(D4-Pad4) -> Net-(R16-Pad1)
- R16 pad 2: /bargraph_driver/L2 -> +5V
- R2 pad 2: Net-(IC1-Pad24) -> Net-(IC1-Pad4)
- R26 pad 1: Net-(R26-Pad1) -> Net-(D14-Pad1)
- R26 pad 2: Net-(D14-Pad1) -> Net-(R26-Pad2)
- R3 pad 2: Net-(IC1-Pad25) -> Net-(IC1-Pad5)
- R4 pad 2: Net-(IC1-Pad26) -> Net-(IC1-Pad6)
- SW3 pad 1: /power rail/BSense -> /BSense
- SW3 pad 2: Net-(D16-Pad1) -> Net-(BT1-Pad1)
- U1 pad 1: +5V -> Net-(R15-Pad1)
- U1 pad 10: /bargraph_driver/S0 -> GND
- U1 pad 11: /bargraph_driver/S1 -> Net-(D4-Pad26)
- U1 pad 12: GND -> Net-(D4-Pad25)
- U1 pad 13: /bargraph_driver/S3 -> Net-(D4-Pad24)
- U1 pad 14: /bargraph_driver/S2 -> Net-(D4-Pad23)
- U1 pad 15: GND -> Net-(D4-Pad22)
- U1 pad 16: Net-(U1-Pad16) -> Net-(D4-Pad21)
- U1 pad 19: Net-(U1-Pad19) -> GND
- U1 pad 2: Net-(D12-Pad1) -> GND
- U1 pad 22: Net-(Q10-Pad1) -> (no net)
- U1 pad 23: Net-(D13-Pad1) -> (no net)
- U1 pad 24: +5V -> GND
- U1 pad 3: Net-(D11-Pad1) -> GND
- U1 pad 4: Net-(D10-Pad1) -> GND
- U1 pad 5: Net-(D9-Pad1) -> GND
- U1 pad 6: Net-(D8-Pad1) -> Net-(D4-Pad30)
- U1 pad 7: Net-(D7-Pad1) -> Net-(D4-Pad29)
- U1 pad 8: Net-(D6-Pad1) -> Net-(D4-Pad28)
- U1 pad 9: Net-(D5-Pad1) -> Net-(D4-Pad27)
- U2 pad 1: Net-(R26-Pad1) -> Net-(R26-Pad2)
Routing:
- net /power rail/BSense: track 49.6 -> 0.00 mm, vias 2 -> 0
- net /bargraph_driver/S3: track 44.1 -> 0.00 mm, vias 1 -> 0
- net Net-(D14-Pad1): track 60.5 -> 19.8 mm, vias 1 -> 0
- net /bargraph_driver/S2: track 38.3 -> 0.00 mm
- net Net-(D13-Pad1): track 37.3 -> 0.00 mm
- net /bargraph_driver/S0: track 32.7 -> 0.00 mm, vias 2 -> 0
- net Net-(Q10-Pad1): track 31.0 -> 0.00 mm
- net Net-(D5-Pad1): track 30.7 -> 0.00 mm
- net /bargraph_driver/S1: track 30.3 -> 0.00 mm, vias 2 -> 0
- net Net-(D7-Pad1): track 24.9 -> 0.00 mm
- net Net-(D11-Pad1): track 23.5 -> 0.00 mm
- net /bargraph_driver/L10: track 22.5 -> 0.00 mm
- net Net-(D9-Pad1): track 22.0 -> 0.00 mm
- net /bargraph_driver/L2: track 21.4 -> 0.00 mm
- net /bargraph_driver/L6: track 20.9 -> 0.00 mm
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