File: KiCad/FencingTester.sch (KiCad schematic (older format))
At the start: 45 parts, among them IC1 ATMEGA328P-P, P1 SERIAL, P2 CONN_01X03, P3 CONN_01X03, SW1 SP3T, SW2 SP3T, Y1 16MHz

Commit message: New bargraph driver + General cleanup
Parts:
- removed R17, R18, R19, R20, R21, R22, R23, R24, R25: 330, Resistors_SMD:R_0805_HandSoldering, symbol Device:R
- added U1: TLC59116, Housings_SSOP:TSSOP-28_4.4x9.7mm_Pitch0.65mm, symbol FencingTester_ComponentsLib:TLC59116
- R15: value 330 -> R
- R16: value 330 -> 10k
Connections:
- net labels added: BSense, SCL, SDA
- wire segments 156 -> 179
- no-connect marks 13 -> 21
Other:
- moved on the sheet: AR1, C1, C2, C3, C4, C5, D1, D2, D3, D4, IC1, R1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

Commit message: i2C
Parts:
- added R? (x2): 10k, symbol Device:R
Connections:
- wire segments 179 -> 187
Changed lines of the file:
@@
 L power:GND #PWR01
 U 1 1 58606032
-P 9350 1900
-F 0 "#PWR01" H 9350 1650 50  0001 C CNN
-F 1 "GND" H 9350 1750 50  0000 C CNN
-F 2 "" H 9350 1900 50  0000 C CNN
-F 3 "" H 9350 1900 50  0000 C CNN
-	1    9350 1900
+P 9450 1900
+F 0 "#PWR01" H 9450 1650 50  0001 C CNN
+F 1 "GND" H 9450 1750 50  0000 C CNN
+F 2 "" H 9450 1900 50  0000 C CNN
+F 3 "" H 9450 1900 50  0000 C CNN
+	1    9450 1900
 	1    0    0    -1
 $EndComp
@@
 Text Label 2950 5250 0    50   ~ 0
 SDA
-Text Label 8350 2450 2    50   ~ 0
+Text Label 9300 2450 2    50   ~ 0
 SDA
-Text Label 8350 2550 2    50   ~ 0
+Text Label 9300 2550 2    50   ~ 0
 SCL
 $Comp
@@
 Wire Wire Line
 	7950 3500 8450 3500
-Wire Wire Line
-	7950 2450 8350 2450
-Wire Wire Line
-	7950 2550 8350 2550
 Wire Wire Line
 	6050 3500 6000 3500
@@
 	9250 1850 9250 2000
 Wire Wire Line
-	9350 1850 9350 1900
-Wire Wire Line
-	9250 1850 9350 1850
+	9450 1850 9450 1900
+Wire Wire Line
+	9250 1850 9450 1850
 Wire Wire Line
 	1500 6300 1700 6300
@@
 	8100 1175 8100 1400
 NoConn ~ 6050 5600
+$Comp
+L Device:R R?
+U 1 1 5BD7E9B3
+P 9250 2300
+F 0 "R?" V 9043 2300 50  0000 C CNN
+F 1 "10k" V 9134 2300 50  0000 C CNN
+F 2 "" V 9180 2300 50  0001 C CNN
+F 3 "~" H 9250 2300 50  0001 C CNN
+	1    9250 2300
+	0    1    1    0
+$EndComp
+$Comp
+L Device:R R?
+U 1 1 5BD94A6A
+P 9250 2700
+F 0 "R?" V 9365 2700 50  0000 C CNN
+F 1 "10k" V 9456 2700 50  0000 C CNN
+F 2 "" V 9180 2700 50  0001 C CNN
+F 3 "~" H 9250 2700 50  0001 C CNN
+	1    9250 2700
+	0    1    1    0
+$EndComp
+Wire Wire Line
+	9400 2300 9450 2300
+Wire Wire Line
+	7950 2550 9050 2550
+Wire Wire Line
+	9100 2700 9050 2700
+Wire Wire Line
+	9050 2700 9050 2550
+Connection ~ 9050 2550
+Wire Wire Line
+	9050 2550 9300 2550
+Wire Wire Line
+	7950 2450 9050 2450
+Wire Wire Line
+	9100 2300 9050 2300
+Wire Wire Line
+	9050 2300 9050 2450
+Connection ~ 9050 2450
+Wire Wire Line
+	9050 2450 9300 2450
+Wire Wire Line
+	9450 2700 9400 2700
+$Comp
+L power:+5V #PWR?
+U 1 1 5BE913A7
+P 9450 2700
+F 0 "#PWR?" H 9450 2550 50  0001 C CNN
+F 1 "+5V" H 9550 2800 50  0000 C CNN
+F 2 "" H 9450 2700 50  0000 C CNN
+F 3 "" H 9450 2700 50  0000 C CNN
+	1    9450 2700
+	1    0    0    -1
+$EndComp
+$Comp
+L power:+5V #PWR?
+U 1 1 5BE91475
+P 9450 2300
+F 0 "#PWR?" H 9450 2150 50  0001 C CNN
+F 1 "+5V" H 9550 2400 50  0000 C CNN
+F 2 "" H 9450 2300 50  0000 C CNN
+F 3 "" H 9450 2300 50  0000 C CNN
+	1    9450 2300
+	1    0    0    -1
+$EndComp
 $EndSCHEMATC

Commit message: Update Schematic
Parts:
- added R17: 330, Resistors_SMD:R_0805_HandSoldering, symbol Device:R
- R15: value R -> 330
- gave numbers to parts that had none: 2
Connections:
- wire segments 187 -> 188
Changed lines of the file:
@@
 P 2750 6100
 F 0 "R15" V 2543 6100 50  0000 C CNN
-F 1 "R" V 2634 6100 50  0000 C CNN
+F 1 "330" V 2634 6100 50  0000 C CNN
 F 2 "Resistors_SMD:R_0805_HandSoldering" V 2680 6100 50  0001 C CNN
 F 3 "~" H 2750 6100 50  0001 C CNN
@@
 Wire Wire Line
 	2600 6100 2550 6100
-Wire Wire Line
-	2550 6100 2550 6200
 $Comp
 L power:GND #PWR0104
 U 1 1 5BF52F54
-P 2550 6200
-F 0 "#PWR0104" H 2550 5950 50  0001 C CNN
-F 1 "GND" H 2555 6027 50  0000 C CNN
-F 2 "" H 2550 6200 50  0001 C CNN
-F 3 "" H 2550 6200 50  0001 C CNN
-	1    2550 6200
+P 2200 6200
+F 0 "#PWR0104" H 2200 5950 50  0001 C CNN
+F 1 "GND" H 2205 6027 50  0000 C CNN
+F 2 "" H 2200 6200 50  0001 C CNN
+F 3 "" H 2200 6200 50  0001 C CNN
+	1    2200 6200
 	1    0    0    -1
 $EndComp
@@
 NoConn ~ 6050 5600
 $Comp
-L Device:R R?
+L Device:R R18
 U 1 1 5BD7E9B3
 P 9250 2300
-F 0 "R?" V 9043 2300 50  0000 C CNN
+F 0 "R18" V 9043 2300 50  0000 C CNN
 F 1 "10k" V 9134 2300 50  0000 C CNN
 F 2 "" V 9180 2300 50  0001 C CNN
@@
 $EndComp
 $Comp
-L Device:R R?
+L Device:R R19
 U 1 1 5BD94A6A
 P 9250 2700
-F 0 "R?" V 9365 2700 50  0000 C CNN
+F 0 "R19" V 9365 2700 50  0000 C CNN
 F 1 "10k" V 9456 2700 50  0000 C CNN
 F 2 "" V 9180 2700 50  0001 C CNN
@@
 	9450 2700 9400 2700
 $Comp
-L power:+5V #PWR?
+L power:+5V #PWR0108
 U 1 1 5BE913A7
 P 9450 2700
-F 0 "#PWR?" H 9450 2550 50  0001 C CNN
+F 0 "#PWR0108" H 9450 2550 50  0001 C CNN
 F 1 "+5V" H 9550 2800 50  0000 C CNN
 F 2 "" H 9450 2700 50  0000 C CNN
@@
 $EndComp
 $Comp
-L power:+5V #PWR?
+L power:+5V #PWR0109
 U 1 1 5BE91475
 P 9450 2300
-F 0 "#PWR?" H 9450 2150 50  0001 C CNN
+F 0 "#PWR0109" H 9450 2150 50  0001 C CNN
 F 1 "+5V" H 9550 2400 50  0000 C CNN
 F 2 "" H 9450 2300 50  0000 C CNN
@@
 	1    0    0    -1
 $EndComp
+$Comp
+L Device:R R17
+U 1 1 5BDE687E
+P 2400 6100
+F 0 "R17" V 2193 6100 50  0000 C CNN
+F 1 "330" V 2284 6100 50  0000 C CNN
+F 2 "Resistors_SMD:R_0805_HandSoldering" V 2330 6100 50  0001 C CNN
+F 3 "~" H 2400 6100 50  0001 C CNN
+	1    2400 6100
+	0    1    1    0
+$EndComp
+Wire Wire Line
+	2250 6100 2200 6100
+Wire Wire Line
+	2200 6100 2200 6200
 $EndSCHEMATC

Commit message: Updating modules libraries
Parts:
- removed P2, P3: CONN_01X03, custom-fencingTester:3PadsWires, symbol conn:CONN_01X03
- added J1, J2: Conn_01x03_Female, custom-fencingTester:3PadsWires, symbol Connector:Conn_01x03_Female
- AR1: footprint Housings_SOIC:SOIC-8_3.9x4.9mm_Pitch1.27mm -> Package_SO:SOIC-8_3.9x4.9mm_P1.27mm
- C1, C2, C3, C4, C5: footprint Capacitors_SMD:C_0805_HandSoldering -> Capacitor_SMD:C_0805_2012Metric_Pad1.15x1.40mm_HandSolder
- IC1: footprint Housings_DIP:DIP-28_W7.62mm_Socket_LongPads -> Package_DIP:DIP-28_W7.62mm_Socket_LongPads
- P1: footprint Pin_Headers:Pin_Header_Straight_1x06_Pitch2.54mm -> Connector_PinHeader_2.54mm:PinHeader_1x06_P2.54mm_Vertical; symbol conn:CONN_01X06 -> FencingTester-rescue:CONN_01X06-conn
- R1, R10, R11, R12, R13, R14, R15, R16, R17, R2, R3, R4, R43, R44, R45, R5, R6, R7, R8, R9: footprint Resistors_SMD:R_0805_HandSoldering -> Resistor_SMD:R_0805_2012Metric_Pad1.15x1.40mm_HandSolder
- R18, R19: footprint (none) -> Resistor_SMD:R_0805_2012Metric_Pad1.15x1.40mm_HandSolder
- U1: footprint Housings_SSOP:TSSOP-28_4.4x9.7mm_Pitch0.65mm -> Package_SO:TSSOP-28_4.4x9.7mm_P0.65mm
