File: KiCad/PowerRail.sch (KiCad schematic (older format))
At the start: 27 parts, among them P4 USB_OTG, Q11 Q_PMOS_DGS, Q12 Q_NMOS_GSD, SW3 SPST, U2 MCP73831, U3 TPS61200

Commit message: Simplifying power rail
We do not switch to USB power anymore when USB is connected
Parts:
- removed C8: 10µF, Capacitors_SMD:C_0805_HandSoldering, symbol Device:C
- removed D16: D_Schottky, Diodes_SMD:SOD-123, symbol Device:D_Schottky
- removed Q11: Q_PMOS_DGS, custom-fencingTester:TSOP-6_HandSoldering, symbol FencingTester-rescue:Q_PMOS_DGS_corrected-RESCUE-FencingTester
- removed Q12: Q_NMOS_GSD, custom-fencingTester:TSMT3, symbol Device:Q_NMOS_GSD
- removed R29: 2k, Resistors_SMD:R_0805_HandSoldering, symbol Device:R
- removed R46: 10k, Resistors_SMD:R_0805_HandSoldering, symbol Device:R
Connections:
- wire segments 57 -> 51
Other:
- moved on the sheet: BT1, C10, C11, C12, C13, C6, C7, D14, P4, R26, R27, R33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

Commit message: Updating modules libraries
Parts:
- C10, C11, C12, C13, C6, C7, C9: footprint Capacitors_SMD:C_0805_HandSoldering -> Capacitor_SMD:C_0805_2012Metric_Pad1.15x1.40mm_HandSolder
- F1: footprint Fuse_Holders_and_Fuses:Fuse_SMD1206_HandSoldering -> Fuse:Fuse_1206_3216Metric_Pad1.42x1.75mm_HandSolder
- R26, R27, R31, R32, R33, R34: footprint Resistors_SMD:R_0805_HandSoldering -> Resistor_SMD:R_0805_2012Metric_Pad1.15x1.40mm_HandSolder
- U2: footprint TO_SOT_Packages_SMD:SOT-23-5 -> Package_TO_SOT_SMD:TSOT-23-5_HandSoldering
Changed lines of the file:
@@
 F 0 "U2" H 3800 3225 60  0000 C CNN
 F 1 "MCP73831" H 3800 4250 60  0000 C CNN
-F 2 "TO_SOT_Packages_SMD:SOT-23-5" H 3800 3750 60  0001 C CNN
+F 2 "Package_TO_SOT_SMD:TSOT-23-5_HandSoldering" H 3800 3750 60  0001 C CNN
 F 3 "" H 3800 3750 60  0000 C CNN
 	1    3800 3750
@@
 F 0 "R26" V 3180 3950 50  0000 C CNN
 F 1 "470" V 3100 3950 50  0000 C CNN
-F 2 "Resistors_SMD:R_0805_HandSoldering" V 3030 3950 50  0001 C CNN
+F 2 "Resistor_SMD:R_0805_2012Metric_Pad1.15x1.40mm_HandSolder" V 3030 3950 50  0001 C CNN
 F 3 "" H 3100 3950 50  0000 C CNN
 	1    3100 3950
@@
 F 0 "C6" H 3325 3500 50  0000 L CNN
 F 1 "4.7µF" H 3075 3300 50  0000 L CNN
-F 2 "Capacitors_SMD:C_0805_HandSoldering" H 3338 3250 50  0001 C CNN
+F 2 "Capacitor_SMD:C_0805_2012Metric_Pad1.15x1.40mm_HandSolder" H 3338 3250 50  0001 C CNN
 F 3 "" H 3300 3400 50  0000 C CNN
 	1    3300 3400
@@
 F 0 "R27" V 4550 3825 50  0000 C CNN
 F 1 "2k" V 4450 3850 50  0000 C CNN
-F 2 "Resistors_SMD:R_0805_HandSoldering" V 4380 3850 50  0001 C CNN
+F 2 "Resistor_SMD:R_0805_2012Metric_Pad1.15x1.40mm_HandSolder" V 4380 3850 50  0001 C CNN
 F 3 "" H 4450 3850 50  0000 C CNN
 	1    4450 3850
@@
 F 0 "C7" H 4625 3800 50  0000 L CNN
 F 1 "4.7µF" H 4625 3600 50  0000 L CNN
-F 2 "Capacitors_SMD:C_0805_HandSoldering" H 4638 3550 50  0001 C CNN
+F 2 "Capacitor_SMD:C_0805_2012Metric_Pad1.15x1.40mm_HandSolder" H 4638 3550 50  0001 C CNN
 F 3 "" H 4600 3700 50  0000 C CNN
 	1    4600 3700
@@
 F 0 "F1" V 7075 3575 50  0000 C CNN
 F 1 "FUSE" V 6900 3475 50  0000 C CNN
-F 2 "Fuse_Holders_and_Fuses:Fuse_SMD1206_HandSoldering" H 7000 3550 50  0001 C CNN
+F 2 "Fuse:Fuse_1206_3216Metric_Pad1.42x1.75mm_HandSolder" H 7000 3550 50  0001 C CNN
 F 3 "" H 7000 3550 50  0000 C CNN
 	1    7000 3550
@@
 F 0 "C9" H 7650 3325 50  0000 L CNN
 F 1 "10µF" H 7600 3500 50  0000 L CNN
-F 2 "Capacitors_SMD:C_0805_HandSoldering" H 7638 3250 50  0001 C CNN
+F 2 "Capacitor_SMD:C_0805_2012Metric_Pad1.15x1.40mm_HandSolder" H 7638 3250 50  0001 C CNN
 F 3 "" H 7600 3400 50  0000 C CNN
 	1    7600 3400
@@
 F 0 "R33" V 9480 3800 50  0000 C CNN
 F 1 "2.4M" V 9400 3800 50  0000 C CNN
-F 2 "Resistors_SMD:R_0805_HandSoldering" V 9330 3800 50  0001 C CNN
+F 2 "Resistor_SMD:R_0805_2012Metric_Pad1.15x1.40mm_HandSolder" V 9330 3800 50  0001 C CNN
 F 3 "" H 9400 3800 50  0000 C CNN
 	1    9400 3800
@@
 F 0 "R34" V 9480 4100 50  0000 C CNN
 F 1 "267k" V 9400 4100 50  0000 C CNN
-F 2 "Resistors_SMD:R_0805_HandSoldering" V 9330 4100 50  0001 C CNN
+F 2 "Resistor_SMD:R_0805_2012Metric_Pad1.15x1.40mm_HandSolder" V 9330 4100 50  0001 C CNN
 F 3 "" H 9400 4100 50  0000 C CNN
 	1    9400 4100
@@
 F 0 "C10" H 9175 4350 50  0000 L CNN
 F 1 "100nF" H 8900 4150 50  0000 L CNN
-F 2 "Capacitors_SMD:C_0805_HandSoldering" H 9188 4100 50  0001 C CNN
+F 2 "Capacitor_SMD:C_0805_2012Metric_Pad1.15x1.40mm_HandSolder" H 9188 4100 50  0001 C CNN
 F 3 "" H 9150 4250 50  0000 C CNN
 	1    9150 4250
@@
 F 0 "C11" H 9775 3900 50  0000 L CNN
 F 1 "10µF" H 9775 3700 50  0000 L CNN
-F 2 "Capacitors_SMD:C_0805_HandSoldering" H 9788 3650 50  0001 C CNN
+F 2 "Capacitor_SMD:C_0805_2012Metric_Pad1.15x1.40mm_HandSolder" H 9788 3650 50  0001 C CNN
 F 3 "" H 9750 3800 50  0000 C CNN
 	1    9750 3800
@@
 F 0 "R31" V 7680 3700 50  0000 C CNN
 F 1 "2.4M" V 7600 3700 50  0000 C CNN
-F 2 "Resistors_SMD:R_0805_HandSoldering" V 7530 3700 50  0001 C CNN
+F 2 "Resistor_SMD:R_0805_2012Metric_Pad1.15x1.40mm_HandSolder" V 7530 3700 50  0001 C CNN
 F 3 "" H 7600 3700 50  0000 C CNN
 	1    7600 3700
@@
 F 0 "R32" V 7675 4000 50  0000 C CNN
 F 1 "220k" V 7600 4000 50  0000 C CNN
-F 2 "Resistors_SMD:R_0805_HandSoldering" V 7530 4000 50  0001 C CNN
+F 2 "Resistor_SMD:R_0805_2012Metric_Pad1.15x1.40mm_HandSolder" V 7530 4000 50  0001 C CNN
 F 3 "" H 7600 4000 50  0000 C CNN
 	1    7600 4000
@@
 F 0 "C12" H 10000 3900 50  0000 L CNN
 F 1 "10µF" H 10000 3700 50  0000 L CNN
-F 2 "Capacitors_SMD:C_0805_HandSoldering" H 10013 3650 50  0001 C CNN
+F 2 "Capacitor_SMD:C_0805_2012Metric_Pad1.15x1.40mm_HandSolder" H 10013 3650 50  0001 C CNN
 F 3 "" H 9975 3800 50  0000 C CNN
 	1    9975 3800
@@
 F 0 "C13" H 7275 3800 50  0000 L CNN
 F 1 "0.1µF" H 7175 3625 50  0000 L CNN
-F 2 "Capacitors_SMD:C_0805_HandSoldering" H 7438 3550 50  0001 C CNN
+F 2 "Capacitor_SMD:C_0805_2012Metric_Pad1.15x1.40mm_HandSolder" H 7438 3550 50  0001 C CNN
 F 3 "" H 7400 3700 50  0001 C CNN
 	1    7400 3700
